Commit message: Add shooter servos and wheels

File: description/inertia.xacro (robot description, xacro)
@@ -1,4 +1,13 @@
 <?xml version="1.0"?>
 <robot xmlns:xacro="http://www.ros.org/wiki/xacro" >
+  <xacro:macro name="inertial_box" params="mass x y z *origin">
+      <inertial>
+          <xacro:insert_block name="origin"/>
+          <mass value="${mass}" />
+          <inertia ixx="${(1/12) * mass * (y*y+z*z)}" ixy="0.0" ixz="0.0"
+                  iyy="${(1/12) * mass * (x*x+z*z)}" iyz="0.0"
+                  izz="${(1/12) * mass * (x*x+y*y)}" />
+      </inertial>
+  </xacro:macro>
   <xacro:macro name="inertial_cylinder" params="mass length radius *origin">
     <inertial>

File: description/robot_core.urdf.xacro (robot description, xacro)
@@ -71,4 +71,66 @@
   <xacro:wheel_macro prefix="FR_wheel" parent="chassis" xyz="0.11829359 -0.11703082 0" rpy="${pi/2} 0 0" axis="0 0 -1"/>
   <xacro:wheel_macro prefix="BR_wheel" parent="chassis" xyz="-0.11829359 -0.11703082 0" rpy="${pi/2} 0 0" axis="0 0 -1"/>
+  <joint name="yaw_shooter_servo_joint" type="revolute">
+    <origin xyz="0 0 0.0633" rpy="0 0 0"/>
+    <parent link="chassis"/>
+    <child  link="shooter_base"/>
+    <axis xyz="0 0 1"/>
+    <limit lower="0" upper="3.49066" velocity="5.5" effort="3.2"/>
+  </joint>
+  <link name="shooter_base">
+    <visual>
+      <geometry>
+        <cylinder length="0.03" radius="0.075"/>
+      </geometry>
+      <material name="red"/>
+    </visual>
+    <collision>
+      <geometry>
+        <cylinder length="0.03" radius="0.075"/>
+      </geometry>
+    </collision>
+    <!-- Please change mass... -->
+    <xacro:inertial_cylinder mass="1" length="0.03" radius="0.075">
+      <origin xyz="0 0 0" rpy="0 0 0"/>
+    </xacro:inertial_cylinder>
+  </link>
+  <joint name="pitch_shooter_servo_joint" type="revolute">
+    <origin xyz="0 0 0.030" rpy="0 0 0"/>
+    <parent link="shooter_base"/>
+    <child link="shooter_body"/>
+    <axis xyz="0 -1 0"/>
+    <limit lower="0" upper="1.0" velocity="3.0" effort="2.0"/>
+  </joint>
+  <link name="shooter_body">
+    <visual>
+      <geometry><box size="0.12 0.04 0.04"/></geometry>
+      <origin xyz="0.06 0 0"/>
+      <material name="blue"/>
+    </visual>
+  </link>
+  <joint name="left_shooter_wheel_joint" type="continuous">
+    <origin xyz="0.12 0.03 0" rpy="-${pi/2} 0 0"/>
+    <parent link="shooter_body"/>
+    <child link="left_wheel"/>
+    <axis xyz="0 0 1"/>
+  </joint>
+  <link name="left_wheel">
+    <visual>
+      <geometry><cylinder length="0.02" radius="0.02"/></geometry>
+      <material name="red"/>
+    </visual>
+  </link>
+  <joint name="right_shooter_wheel_joint" type="continuous">
+    <origin xyz="0.12 -0.03 0" rpy="${pi/2} 0 0"/>
+    <parent link="shooter_body"/>
+    <child link="right_wheel"/>
+    <axis xyz="0 0 -1"/>
+  </joint>
+  <link name="right_wheel">
+    <visual>
+      <geometry><cylinder length="0.02" radius="0.02"/></geometry>
+      <material name="red"/>
+    </visual>
+  </link>
   <!-- <joint name="camera_joint" type="fixed"> -->
   <!--   <parent link="base_link"/> -->

File: description/ros2_control.xacro (robot description, xacro)
@@ -45,14 +45,15 @@
           <param name="BR_wheel_name">BR_wheel_joint</param>
           <param name="FR_wheel_name">FR_wheel_joint</param>
-          <param name="loop_rate">30</param>
+          <param name="left_shooter_wheel_name">left_shooter_wheel_joint</param>
+          <param name="right_shooter_wheel_name">right_shooter_wheel_joint</param>
+          <param name="enc_counts_per_rev">3436</param>
+          <param name="yaw_shooter_servo_name">yaw_shooter_servo_joint</param>
+          <param name="pitch_shooter_servo_name">pitch_shooter_servo_joint</param>
           <param name="device">/dev/ttyACM0</param>
           <param name="baud_rate">115200</param>
+          <param name="loop_rate">30</param>
           <param name="timeout_ms">1000</param>
-          <param name="enc_counts_per_rev">3436</param>
-          <param name="pid_p">20</param>
-          <param name="pid_d">12</param>
-          <param name="pid_i">0</param>
-          <param name="pid_o">50</param>
         </hardware>
+        <!-- Drive  -->
         <joint name="FL_wheel_joint">
           <command_interface name="velocity">
@@ -87,4 +88,21 @@
           <state_interface name="velocity"/>
         </joint>
+        <!-- Shooter -->
+        <joint name="left_shooter_wheel_joint">
+          <command_interface name="velocity"/>
+          <state_interface name="velocity"/>
+        </joint>
+        <joint name="right_shooter_wheel_joint">
+          <command_interface name="velocity"/>
+          <state_interface name="velocity"/>
+        </joint>
+        <joint name="yaw_shooter_servo_joint">
+          <command_interface name="position"/>
+          <state_interface name="position"/>
+        </joint>
+        <joint name="pitch_shooter_servo_joint">
+          <command_interface name="position"/>
+          <state_interface name="position"/>
+        </joint>
       </ros2_control>
     </xacro:unless>
