Commit message: Add pose for targets and apriltags

File: description/ros2_control.xacro (robot description, xacro)
@@ -50,4 +50,7 @@
           <param name="yaw_shooter_servo_name">yaw_shooter_servo_joint</param>
           <param name="pitch_shooter_servo_name">pitch_shooter_servo_joint</param>
+          <param name="intake_servo_name">intake_servo_joint</param>
+          <param name="intake_wheel_name">intake_wheel_joint</param>
+          <param name="stick_servo_name">stick_servo_joint</param>
           <param name="device">/dev/ttyACM0</param>
           <param name="baud_rate">115200</param>
@@ -105,4 +108,18 @@
           <state_interface name="position"/>
         </joint>
+	<!-- Intake -->
+        <joint name="intake_servo_joint">
+          <command_interface name="position"/>
+          <state_interface name="position"/>
+        </joint>
+        <joint name="intake_wheel_joint">
+          <command_interface name="velocity"/>
+          <state_interface name="velocity"/>
+        </joint>
+	<!-- Stick -->
+        <joint name="stick_servo_joint">
+          <command_interface name="position"/>
+          <state_interface name="position"/>
+        </joint>
       </ros2_control>
     </xacro:unless>
