Commit message: Add final robot design as urdf

File: description/robot.urdf.xacro (robot description, xacro)
@@ -1,9 +1,8 @@
 <?xml version="1.0"?>
 <robot xmlns:xacro="http://www.ros.org/wiki/xacro" name="robot">
-  <xacro:arg name="prefix" default=""/>
   <xacro:arg name="sim_mode" default="false"/>
   <xacro:include filename="robot_core.urdf.xacro"/>
   <xacro:include filename="ros2_control.xacro" />
-  <xacro:robot prefix="$(arg prefix)" sim_mode="$(arg sim_mode)"/>
-  <xacro:robot_control name="robot" prefix="$(arg prefix)" sim_mode="$(arg sim_mode)" />
+  <xacro:robot_core sim_mode="$(arg sim_mode)"/>
+  <xacro:robot_control sim_mode="$(arg sim_mode)" />
 </robot>

File: description/robot_core.urdf.xacro (robot description, xacro)
@@ -1,151 +1,5761 @@
 <?xml version="1.0" ?>
 <robot xmlns:xacro="http://www.ros.org/wiki/xacro">
-  <xacro:macro name="robot" params="prefix sim_mode:=false">
-  <xacro:include filename="inertia.xacro"/>
-  <material name="blue">
-    <color rgba="0 0 1.0 1.0"/>
-  </material>
-  <material name="green">
-    <color rgba="0 1.0 0 1.0"/>
-  </material>
-  <material name="red">
-    <color rgba="1.0 0 0 1.0"/>
-  </material>
-  <!-- This macro will make life easier. Source: trust me bro -->
-  <xacro:macro name="wheel_macro" params="parent prefix xyz rpy axis">
-    <joint name="${prefix}_joint" type="continuous">
-      <origin xyz="${xyz}" rpy="${rpy}"/>
-      <parent link="${parent}"/>
-      <child  link="${prefix}_link"/>
-      <axis xyz="${axis}"/>
-    </joint>
-    <link name="${prefix}_link">
-      <visual>
-        <geometry>
-          <cylinder length="0.03643720" radius="0.035369"/>
-        </geometry>
-        <material name="red"/>
-      </visual>
-      <collision>
-        <geometry>
-          <sphere radius="0.035369"/>
-        </geometry>
-      </collision>
-      <!-- Please change mass... -->
-      <xacro:inertial_cylinder mass="1" length="0.03643720" radius="0.035369">
-        <origin xyz="0 0 0" rpy="0 0 0"/>
-      </xacro:inertial_cylinder>
-    </link>
-  </xacro:macro>
-  <link name="base_link"/>
-  <joint name="chassis_joint" type="fixed">
+  <xacro:macro name="robot_core" params="sim_mode">
+  <link name="base_link"></link>
+  <joint name="coc_dt_joint" type="fixed">
     <parent link="base_link"/>
-    <child link="chassis"/>
+    <child link="coc_dt"/>
     <origin xyz="0 0 0"/>
   </joint>
-  <link name="chassis">
+  <link name="coc_dt">
     <inertial>
-      <origin xyz="3.84321e-10 9.33138e-10 0.0163291" rpy="0 0 -${pi/2}"/>
-      <!-- Please change mass and inertia matrix to reflect better aprox -->
-      <mass value="16.479"/>
-      <inertia ixx="0.174135" ixy="1.42629e-09" ixz="-7.38887e-11" iyy="0.119734" iyz="-1.54691e-10" izz="0.279608"/>
+      <origin xyz="0 0 0" rpy="0 0 0"/>
+      <mass value="1e-09"/>
+      <inertia ixx="1e-09" ixy="0" ixz="0" iyy="1e-09" iyz="0" izz="1e-09"/>
     </inertial>
-    <visual>
-      <origin xyz="0 0 0" rpy="0 -0 -${pi/2}"/>
-      <geometry>
-        <mesh filename="package://rivals/description/assets/part_1__6ed075fc00e4d09673dc30a20c0a2d67.stl"/>
-      </geometry>
-      <material name="part_1__6ed075fc00e4d09673dc30a20c0a2d67_material">
+    <!-- Part hex_socket_head_cap_screw_m3x0_50_x_14 -->
+    <visual>
+      <origin xyz="-0.100404 0.089725 0.003" rpy="0 -0 -1.5708"/>
+      <geometry>
+        <mesh filename="package://rivals/description/assets/hex_socket_head_cap_screw_m3x0_50_x_14.stl"/>
+      </geometry>
+      <material name="hex_socket_head_cap_screw_m3x0_50_x_14_material">
+        <color rgba="0.603922 0.647059 0.686275 1"/>
+      </material>
+    </visual>
+    <collision>
+      <origin xyz="-0.100404 0.089725 0.003" rpy="0 -0 -1.5708"/>
+      <geometry>
+        <mesh filename="package://rivals/description/assets/hex_socket_head_cap_screw_m3x0_50_x_14.stl"/>
+      </geometry>
+    </collision>
+    <!-- Part hex_socket_head_cap_screw_m3x0_50_x_14_2 -->
+    <visual>
+      <origin xyz="-0.132404 -0.089725 0.003" rpy="0 -0 -1.5708"/>
+      <geometry>
+        <mesh filename="package://rivals/description/assets/hex_socket_head_cap_screw_m3x0_50_x_14.stl"/>
+      </geometry>
+      <material name="hex_socket_head_cap_screw_m3x0_50_x_14_2_material">
+        <color rgba="0.603922 0.647059 0.686275 1"/>
+      </material>
+    </visual>
+    <collision>
+      <origin xyz="-0.132404 -0.089725 0.003" rpy="0 -0 -1.5708"/>
+      <geometry>
+        <mesh filename="package://rivals/description/assets/hex_socket_head_cap_screw_m3x0_50_x_14.stl"/>
+      </geometry>
+    </collision>
+    <!-- Part part_61 -->
+    <visual>
+      <origin xyz="-6.31296e-17 0 -0.056493" rpy="0 -0 -1.5708"/>
+      <geometry>
+        <mesh filename="package://rivals/description/assets/part_61.stl"/>
+      </geometry>
+      <material name="part_61_material">
+        <color rgba="0.768627 0.886275 0.952941 1"/>
+      </material>
+    </visual>
+    <collision>
+      <origin xyz="-6.31296e-17 0 -0.056493" rpy="0 -0 -1.5708"/>
+      <geometry>
+        <mesh filename="package://rivals/description/assets/part_61.stl"/>
+      </geometry>
+    </collision>
+    <!-- Part hex_socket_head_cap_screw_m3x0_50_x_10 -->
+    <visual>
+      <origin xyz="0.0838042 -0.165497 0.0132894" rpy="0.523599 -0 -1.5708"/>
+      <geometry>
+        <mesh filename="package://rivals/description/assets/hex_socket_head_cap_screw_m3x0_50_x_10.stl"/>
+      </geometry>
+      <material name="hex_socket_head_cap_screw_m3x0_50_x_10_material">
+        <color rgba="0.603922 0.647059 0.686275 1"/>
+      </material>
+    </visual>
+    <collision>
+      <origin xyz="0.0838042 -0.165497 0.0132894" rpy="0.523599 -0 -1.5708"/>
+      <geometry>
+        <mesh filename="package://rivals/description/assets/hex_socket_head_cap_screw_m3x0_50_x_10.stl"/>
+      </geometry>
+    </collision>
+    <!-- Part hex_socket_head_cap_screw_m3x0_50_x_10_2 -->
+    <visual>
+      <origin xyz="-0.1016 -0.1016 0.00735" rpy="0 -0 -1.5708"/>
+      <geometry>
+        <mesh filename="package://rivals/description/assets/hex_socket_head_cap_screw_m3x0_50_x_10.stl"/>
+      </geometry>
+      <material name="hex_socket_head_cap_screw_m3x0_50_x_10_2_material">
+        <color rgba="0.603922 0.647059 0.686275 1"/>
+      </material>
+    </visual>
+    <collision>
+      <origin xyz="-0.1016 -0.1016 0.00735" rpy="0 -0 -1.5708"/>
+      <geometry>
+        <mesh filename="package://rivals/description/assets/hex_socket_head_cap_screw_m3x0_50_x_10.stl"/>
+      </geometry>
+    </collision>
+    <!-- Part 608_2rs -->
+    <visual>
+      <origin xyz="-6.31296e-17 0 -0.056493" rpy="0 -0 -1.5708"/>
+      <geometry>
+        <mesh filename="package://rivals/description/assets/608_2rs.stl"/>
+      </geometry>
+      <material name="608_2rs_material">
+        <color rgba="0.682353 0.333333 0.737255 1"/>
+      </material>
+    </visual>
+    <collision>
+      <origin xyz="-6.31296e-17 0 -0.056493" rpy="0 -0 -1.5708"/>
+      <geometry>
+        <mesh filename="package://rivals/description/assets/608_2rs.stl"/>
+      </geometry>
+    </collision>
+    <!-- Part gt2_3mm_550_motor_pinion_pulley___12_tooth__rev_21_1908 -->
+    <visual>
+      <origin xyz="-6.31296e-17 0 -0.056493" rpy="0 -0 -1.5708"/>
+      <geometry>
+        <mesh filename="package://rivals/description/assets/gt2_3mm_550_motor_pinion_pulley___12_tooth__rev_21_1908.stl"/>
+      </geometry>
+      <material name="gt2_3mm_550_motor_pinion_pulley___12_tooth__rev_21_1908_material">
+        <color rgba="0.12549 0.12549 0.12549 1"/>
+      </material>
+    </visual>
+    <collision>
+      <origin xyz="-6.31296e-17 0 -0.056493" rpy="0 -0 -1.5708"/>
+      <geometry>
+        <mesh filename="package://rivals/description/assets/gt2_3mm_550_motor_pinion_pulley___12_tooth__rev_21_1908.stl"/>
+      </geometry>
+    </collision>
+    <!-- Part batbox -->
+    <visual>
+      <origin xyz="-6.31296e-17 0 -0.056493" rpy="0 -0 -1.5708"/>
+      <geometry>
+        <mesh filename="package://rivals/description/assets/batbox.stl"/>
+      </geometry>
+      <material name="batbox_material">
+        <color rgba="0.231373 0.380392 0.705882 1"/>
+      </material>
+    </visual>
+    <collision>
+      <origin xyz="-6.31296e-17 0 -0.056493" rpy="0 -0 -1.5708"/>
+      <geometry>
+        <mesh filename="package://rivals/description/assets/batbox.stl"/>
+      </geometry>
+    </collision>
+    <!-- Part hex_socket_head_cap_screw_m3x0_50_x_10_3 -->
+    <visual>
+      <origin xyz="0.0508 -0.1016 0.008525" rpy="0 -0 -1.5708"/>
+      <geometry>
+        <mesh filename="package://rivals/description/assets/hex_socket_head_cap_screw_m3x0_50_x_10.stl"/>
+      </geometry>
+      <material name="hex_socket_head_cap_screw_m3x0_50_x_10_3_material">
+        <color rgba="0.603922 0.647059 0.686275 1"/>
+      </material>
+    </visual>
+    <collision>
+      <origin xyz="0.0508 -0.1016 0.008525" rpy="0 -0 -1.5708"/>
+      <geometry>
+        <mesh filename="package://rivals/description/assets/hex_socket_head_cap_screw_m3x0_50_x_10.stl"/>
+      </geometry>
+    </collision>
+    <!-- Part gt2_3mm_550_motor_pinion_pulley___12_tooth__rev_21_1908_2 -->
+    <visual>
+      <origin xyz="-6.31296e-17 0 -0.056493" rpy="0 -0 -1.5708"/>
+      <geometry>
+        <mesh filename="package://rivals/description/assets/gt2_3mm_550_motor_pinion_pulley___12_tooth__rev_21_1908__2.stl"/>
+      </geometry>
+      <material name="gt2_3mm_550_motor_pinion_pulley___12_tooth__rev_21_1908_2_material">
+        <color rgba="0.12549 0.12549 0.12549 1"/>
+      </material>
+    </visual>
+    <collision>
+      <origin xyz="-6.31296e-17 0 -0.056493" rpy="0 -0 -1.5708"/>
+      <geometry>
+        <mesh filename="package://rivals/description/assets/gt2_3mm_550_motor_pinion_pulley___12_tooth__rev_21_1908__2.stl"/>
+      </geometry>
+    </collision>
+    <!-- Part hex_socket_head_cap_screw_m3x0_50_x_14_3 -->
+    <visual>
+      <origin xyz="0.148404 0.089725 0.003" rpy="0 -0 -1.5708"/>
+      <geometry>
+        <mesh filename="package://rivals/description/assets/hex_socket_head_cap_screw_m3x0_50_x_14.stl"/>
+      </geometry>
+      <material name="hex_socket_head_cap_screw_m3x0_50_x_14_3_material">
+        <color rgba="0.603922 0.647059 0.686275 1"/>
+      </material>
+    </visual>
+    <collision>
+      <origin xyz="0.148404 0.089725 0.003" rpy="0 -0 -1.5708"/>
+      <geometry>
+        <mesh filename="package://rivals/description/assets/hex_socket_head_cap_screw_m3x0_50_x_14.stl"/>
+      </geometry>
+    </collision>
+    <!-- Part 608_2rs_2 -->
+    <visual>
+      <origin xyz="-6.31296e-17 0 -0.056493" rpy="0 -0 -1.5708"/>
+      <geometry>
+        <mesh filename="package://rivals/description/assets/608_2rs__2.stl"/>
+      </geometry>
+      <material name="608_2rs_2_material">
+        <color rgba="0.682353 0.333333 0.737255 1"/>
+      </material>
+    </visual>
+    <collision>
+      <origin xyz="-6.31296e-17 0 -0.056493" rpy="0 -0 -1.5708"/>
+      <geometry>
+        <mesh filename="package://rivals/description/assets/608_2rs__2.stl"/>
+      </geometry>
+    </collision>
+    <!-- Part part_30 -->
+    <visual>
+      <origin xyz="-6.31296e-17 0 -0.056493" rpy="0 -0 -1.5708"/>
+      <geometry>
+        <mesh filename="package://rivals/description/assets/part_30.stl"/>
+      </geometry>
+      <material name="part_30_material">
+        <color rgba="0.917647 0.917647 0.917647 1"/>
+      </material>
+    </visual>
+    <collision>
+      <origin xyz="-6.31296e-17 0 -0.056493" rpy="0 -0 -1.5708"/>
+      <geometry>
+        <mesh filename="package://rivals/description/assets/part_30.stl"/>
+      </geometry>
+    </collision>
+    <!-- Part hex_socket_head_cap_screw_m3x0_50_x_30_x_18 -->
+    <visual>
+      <origin xyz="-0.0697334 -0.07955 -0.0149052" rpy="-1.5708 -0 0"/>
+      <geometry>
+        <mesh filename="package://rivals/description/assets/hex_socket_head_cap_screw_m3x0_50_x_30_x_18.stl"/>
+      </geometry>
+      <material name="hex_socket_head_cap_screw_m3x0_50_x_30_x_18_material">
+        <color rgba="0.603922 0.647059 0.686275 1"/>
+      </material>
+    </visual>
+    <collision>
+      <origin xyz="-0.0697334 -0.07955 -0.0149052" rpy="-1.5708 -0 0"/>
+      <geometry>
+        <mesh filename="package://rivals/description/assets/hex_socket_head_cap_screw_m3x0_50_x_30_x_18.stl"/>
+      </geometry>
+    </collision>
+    <!-- Part hex_socket_head_cap_screw_m3x0_50_x_14_4 -->
+    <visual>
+      <origin xyz="0.132404 0.089725 0.003" rpy="0 -0 -1.5708"/>
+      <geometry>
+        <mesh filename="package://rivals/description/assets/hex_socket_head_cap_screw_m3x0_50_x_14.stl"/>
+      </geometry>
+      <material name="hex_socket_head_cap_screw_m3x0_50_x_14_4_material">
+        <color rgba="0.603922 0.647059 0.686275 1"/>
+      </material>
+    </visual>
+    <collision>
+      <origin xyz="0.132404 0.089725 0.003" rpy="0 -0 -1.5708"/>
+      <geometry>
+        <mesh filename="package://rivals/description/assets/hex_socket_head_cap_screw_m3x0_50_x_14.stl"/>
+      </geometry>
+    </collision>
+    <!-- Part hex_socket_head_cap_screw_m3x0_50_x_10_4 -->
+    <visual>
+      <origin xyz="0.157788 -0.0140388 -0.043793" rpy="1.5708 -0 -0.785398"/>
+      <geometry>
+        <mesh filename="package://rivals/description/assets/hex_socket_head_cap_screw_m3x0_50_x_10.stl"/>
+      </geometry>
+      <material name="hex_socket_head_cap_screw_m3x0_50_x_10_4_material">
+        <color rgba="0.603922 0.647059 0.686275 1"/>
+      </material>
+    </visual>
+    <collision>
+      <origin xyz="0.157788 -0.0140388 -0.043793" rpy="1.5708 -0 -0.785398"/>
+      <geometry>
+        <mesh filename="package://rivals/description/assets/hex_socket_head_cap_screw_m3x0_50_x_10.stl"/>
+      </geometry>
+    </collision>
+    <!-- Part hex_socket_head_cap_screw_m3x0_50_x_30_x_18_2 -->
+    <visual>
+      <origin xyz="0.0526581 -0.07955 -0.0194805" rpy="-1.5708 -0 0"/>
+      <geometry>
+        <mesh filename="package://rivals/description/assets/hex_socket_head_cap_screw_m3x0_50_x_30_x_18.stl"/>
+      </geometry>
+      <material name="hex_socket_head_cap_screw_m3x0_50_x_30_x_18_2_material">
+        <color rgba="0.603922 0.647059 0.686275 1"/>
+      </material>
+    </visual>
+    <collision>
+      <origin xyz="0.0526581 -0.07955 -0.0194805" rpy="-1.5708 -0 0"/>
+      <geometry>
+        <mesh filename="package://rivals/description/assets/hex_socket_head_cap_screw_m3x0_50_x_30_x_18.stl"/>
+      </geometry>
+    </collision>
+    <!-- Part hex_socket_head_cap_screw_m3x0_50_x_14_5 -->
+    <visual>
+      <origin xyz="0.1324 0.145225 0.003" rpy="0 -0 -1.5708"/>
+      <geometry>
+        <mesh filename="package://rivals/description/assets/hex_socket_head_cap_screw_m3x0_50_x_14.stl"/>
+      </geometry>
+      <material name="hex_socket_head_cap_screw_m3x0_50_x_14_5_material">
+        <color rgba="0.603922 0.647059 0.686275 1"/>
+      </material>
+    </visual>
+    <collision>
+      <origin xyz="0.1324 0.145225 0.003" rpy="0 -0 -1.5708"/>
+      <geometry>
+        <mesh filename="package://rivals/description/assets/hex_socket_head_cap_screw_m3x0_50_x_14.stl"/>
+      </geometry>
+    </collision>
+    <!-- Part grommet -->
+    <visual>
+      <origin xyz="-6.31296e-17 0 -0.056493" rpy="0 -0 -1.5708"/>
+      <geometry>
+        <mesh filename="package://rivals/description/assets/grommet.stl"/>
+      </geometry>
+      <material name="grommet_material">
         <color rgba="0.615686 0.811765 0.929412 1"/>
       </material>
     </visual>
     <collision>
-      <origin xyz="0 0 0" rpy="0 -0 -${pi/2}"/>
-      <geometry>
-        <mesh filename="package://rivals/description/assets/part_1__6ed075fc00e4d09673dc30a20c0a2d67.stl"/>
+      <origin xyz="-6.31296e-17 0 -0.056493" rpy="0 -0 -1.5708"/>
+      <geometry>
+        <mesh filename="package://rivals/description/assets/grommet.stl"/>
+      </geometry>
+    </collision>
+    <!-- Part smaller550spacer -->
+    <visual>
+      <origin xyz="-6.31296e-17 0 -0.056493" rpy="0 -0 -1.5708"/>
+      <geometry>
+        <mesh filename="package://rivals/description/assets/smaller550spacer.stl"/>
+      </geometry>
+      <material name="smaller550spacer_material">
+        <color rgba="0.596078 0.121569 0.67451 1"/>
+      </material>
+    </visual>
+    <collision>
+      <origin xyz="-6.31296e-17 0 -0.056493" rpy="0 -0 -1.5708"/>
+      <geometry>
+        <mesh filename="package://rivals/description/assets/smaller550spacer.stl"/>
+      </geometry>
+    </collision>
+    <!-- Part hex_socket_head_cap_screw_m3x0_50_x_30_x_18_3 -->
+    <visual>
+      <origin xyz="0.0697334 -0.07955 -0.0149052" rpy="-1.5708 -0 0"/>
+      <geometry>
+        <mesh filename="package://rivals/description/assets/hex_socket_head_cap_screw_m3x0_50_x_30_x_18.stl"/>
+      </geometry>
+      <material name="hex_socket_head_cap_screw_m3x0_50_x_30_x_18_3_material">
+        <color rgba="0.603922 0.647059 0.686275 1"/>
+      </material>
+    </visual>
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
File: description/ros2_control.xacro (robot description, xacro)
@@ -1,5 +1,6 @@
 <?xml version="1.0"?>
 <robot xmlns:xacro="http://www.ros.org/wiki/xacro">
-  <xacro:macro name="robot_control" params="name prefix sim_mode:=false">
+  <xacro:macro name="robot_control" params="sim_mode">
+    <!-- TODO: Haven't got the chance to add the new joints for sim mode :( -->
     <xacro:if value="${sim_mode}">
       <!-- Want Isaac to consume the joint speeds not /cmd_vel -->
@@ -108,5 +109,5 @@
           <state_interface name="position"/>
         </joint>
-	<!-- Intake -->
+        <!-- Intake -->
         <joint name="intake_servo_joint">
           <command_interface name="position"/>
@@ -117,5 +118,5 @@
           <state_interface name="velocity"/>
         </joint>
-	<!-- Stick -->
+        <!-- Stick -->
         <joint name="stick_servo_joint">
           <command_interface name="position"/>
